File: PCBFiles+Schematics/Main PCB/info_orbs.kicad_pcb (KiCad board)
At the start: 2 copper layers, 198.8 x 28.5 mm, 12 parts

Commit message: Updated New PCB Files
Parts:
- added G***: LOGO, A Local Libs:cap, B.Cu at (131.2, 62.8)
- added G***: LOGO, A Local Libs:Untitled, B.Cu at (134.3, 62.7)
- added J1: Conn_01x02_Pin, Connector_PinHeader_2.54mm:PinHeader_1x02_P2.54mm_Vertical, F.Cu at (133.9, 65.9)
- added V2: ESP32-DEVKITC-32D, A Local Libs:38 Pin Board thin, B.Cu at (73.0, 78.1)
- USBPower1: renamed from USB C
- renumbered LFT to SW1, OK to SW2, RHT to SW3, D1 to tft1, D2 to tft2, D3 to tft3, D4 to tft4, D5 to tft5
Connections:
- SW1 pad 2: Net-(U1-vcc) -> Net-(U1-3.3v)
- SW2 pad 2: Net-(U1-vcc) -> Net-(U1-3.3v)
- SW3 pad 2: Net-(U1-vcc) -> Net-(U1-3.3v)
- U1 pad 3: Net-(U1-GND) -> Net-(J1-Pin_1)
- USBPower1 pad 4: Net-(USBPower1-GND) -> Net-(J1-Pin_1)
- V1 pad J2-14: Net-(U1-GND) -> Net-(J1-Pin_1)
- V1 pad J2-16: unconnected-(V1-SD2-PadJ2-16) -> Net-(V1-SD2)
- V1 pad J2-17: unconnected-(V1-SD3-PadJ2-17) -> Net-(V1-SD3)
- V1 pad J2-18: unconnected-(V1-CMD-PadJ2-18) -> Net-(V1-CMD)
- V1 pad J2-2: unconnected-(V1-EN-PadJ2-2) -> Net-(J1-Pin_2)
- V1 pad J2-3: unconnected-(V1-SENSOR_VP-PadJ2-3) -> Net-(V1-SENSOR_VP)
- V1 pad J2-4: unconnected-(V1-SENSOR_VN-PadJ2-4) -> Net-(V1-SENSOR_VN)
- V1 pad J3-1: Net-(USBPower1-GND) -> Net-(J1-Pin_1)
- V1 pad J3-10: unconnected-(V1-IO5-PadJ3-10) -> Net-(V1-IO5)
- V1 pad J3-12: unconnected-(V1-IO16-PadJ3-12) -> Net-(V1-IO16)
- V1 pad J3-13: unconnected-(V1-IO4-PadJ3-13) -> Net-(V1-IO4)
- V1 pad J3-14: unconnected-(V1-IO0-PadJ3-14) -> Net-(V1-IO0)
- V1 pad J3-15: unconnected-(V1-IO2-PadJ3-15) -> Net-(V1-IO2)
- V1 pad J3-16: unconnected-(V1-IO15-PadJ3-16) -> Net-(V1-IO15)
- V1 pad J3-17: unconnected-(V1-SD1-PadJ3-17) -> Net-(V1-SD1)
- V1 pad J3-18: unconnected-(V1-SD0-PadJ3-18) -> Net-(V1-SD0)
- V1 pad J3-19: unconnected-(V1-CLK-PadJ3-19) -> Net-(V1-CLK)
- V1 pad J3-3: unconnected-(V1-IO22-PadJ3-3) -> Net-(V1-IO22)
- V1 pad J3-4: unconnected-(V1-TXD0-PadJ3-4) -> Net-(V1-TXD0)
- V1 pad J3-5: unconnected-(V1-RXD0-PadJ3-5) -> Net-(V1-RXD0)
- V1 pad J3-7: Net-(V1-GND2) -> Net-(J1-Pin_1)
- tft1 pad 6: Net-(V1-GND2) -> Net-(J1-Pin_1)
- tft1 pad 7: Net-(U1-vcc) -> Net-(U1-3.3v)
- tft2 pad 6: Net-(V1-GND2) -> Net-(J1-Pin_1)
- tft2 pad 7: Net-(U1-vcc) -> Net-(U1-3.3v)
- tft3 pad 6: Net-(V1-GND2) -> Net-(J1-Pin_1)
- tft3 pad 7: Net-(U1-vcc) -> Net-(U1-3.3v)
- tft4 pad 6: Net-(V1-GND2) -> Net-(J1-Pin_1)
- tft4 pad 7: Net-(U1-vcc) -> Net-(U1-3.3v)
- tft5 pad 6: Net-(V1-GND2) -> Net-(J1-Pin_1)
- tft5 pad 7: Net-(U1-vcc) -> Net-(U1-3.3v)
Routing:
- net Net-(J1-Pin_1): track 0.00 -> 265.9 mm, vias 0 -> 14
- net Net-(V1-GND2): track 222.8 -> 0.00 mm, vias 4 -> 0
- net Net-(U1-3.3v): track 69.8 -> 259.7 mm, vias 0 -> 5
- net Net-(U1-vcc): track 258.6 -> 73.0 mm, vias 9 -> 1
- net Net-(U1-gpio12): track 160.2 -> 31.8 mm, vias 1 -> 0
- net Net-(USBPower1-GND): track 110.0 -> 0.00 mm, vias 1 -> 0
- net Net-(J1-Pin_2): track 0.00 -> 88.6 mm, vias 0 -> 2
- net Net-(V1-IO17): track 219.5 -> 178.6 mm, vias 8 -> 5
- net Net-(U1-GND): track 32.4 -> 0.00 mm
- net Net-(V1-IO19): track 201.5 -> 173.9 mm
- net Net-(V1-IO32): track 93.3 -> 70.7 mm
- net Net-(U1-gpio35): track 83.1 -> 65.5 mm
- net Net-(U1-gipo34): track 53.1 -> 69.2 mm, vias 0 -> 2
- net Net-(V1-IO21): track 163.8 -> 151.5 mm, vias 1 -> 2
- net Net-(V1-IO18): track 184.3 -> 176.3 mm, vias 1 -> 5
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Other:
- board text added: "<- long hold on boot to reset wifi & config"
- board text added: "Built/Contributed to by: Bram Verhulst, Jae Kitchens, Noah Piqué, Eric Thelin, Davemanchap, Daniel Springer, Mark Jansen, lyricnz, Hugobalder, Christian Erpelding, Matthew Anderson, KanyonKris, Petersch, RacingSquirrel, Sjoerd Verweij, Dave Hill, stv0g, RobThree, Ledomme, JulianSelf, cpwillis, Dave Reed"
- board text added: "EN"
- board text added: "Mode"
- board text added: "Next Widget"
- board text added: "Style"
- board text added: "WARNING: BE CAREFUL CLEANING WITH ISOPROPYL, EVEN A SMALL AMOUNT OF FUMES WILL DAMAGE THE SCREENS"
- board text added: "info orbs v0.3"
- board text removed: "5V PIN>"
- board text removed: "Built/Contributed to by: Bram Verhulst, Jae Kitchens, Noah Piqué, Eric Thelin, Davemanchap, Daniel Springer"
- board text removed: "info orbs v0.2"
